File: PCB/Barghest RP2040 Pro Micro by Shrimped.kicad_sch (KiCad schematic)
At the start: 140 parts, among them SW1 RotaryEncoder_Switch, SW2 RotaryEncoder_Switch, SW3 ROT_SKYLOONG_HS, SW4 ROT_SKYLOONG_HS, U1 RP2040_Pro_Micro

Commit message: Fixed Schematic
Uploaded the incorrect schem
Parts:
- removed SW3, SW4: ROT_SKYLOONG_HS, PCM_marbastlib-various:ROT_SKYLOONG_HS-Switch, symbol PCM_marbastlib-various:ROT_SKYLOONG_HS-Switch
- U1: footprint ScottoKeebs_MCU:RP2040_Pro_Micro -> ScottoKeebs_MCU:RP2040_Pro_Micro_Flipped
Connections:
- net COL0 is gone; now on net col11: U1.8 (GP4)
- net COL1 is gone; now on net col10: U1.9 (GP5)
- net COL10 is gone; now on net col1: U1.25 (GP28)
- net COL11 is gone; now on net col0: U1.26 (GP29)
- net COL2 is gone; now on net col9: U1.10 (GP6)
- net COL3 is gone; now on net col8: U1.11 (GP7)
- net COL4 is gone; now on net col7: U1.12 (GP8)
- net COL5 is gone; now on net col6: U1.13 (GP9)
- net COL6 is gone; now on net row2: U1.21 (GP20)
- net COL7 is gone; now on net row3: U1.22 (GP22)
- net COL8 is gone; now on net row4: U1.23 (GP26)
- net COL9 is gone; now on net col2: U1.24 (GP27)
- net ROT0 is gone; now on net ENCB: C24.1, SW1.A
- net ROT1 is gone; now on net ENCA: C25.2, SW1.B
- net ROT2 is gone; now on net ENCA: C26.1, SW2.A
- net ROT3 is gone; now on net ENCB: C27.2, SW2.B
- net ROW1 is gone; now on net col5: U1.14 (GP12)
- net ROW2 is gone; now on net col4: U1.15 (GP13)
- net ROW3 is gone; now on net col3: U1.16 (GP14)
- net ROW0: no longer U1.7 (GP3)
- net col12: now also U1.7 (GP3)
- net col5: now also SW2.S2
- net row0: now also U1.19 (GP21)
- net row1: now also U1.20 (GP23)
- net at SW2.S1: now also D58.2 (A), MX61.2
- net LEDs: no longer names the net of U1.1 (GP10)
Other:
- moved on the sheet: C26, C27, SW2
